Commit message: add packages name_space & debug

File: rby1_moveit/rby1_moveit_a_1_0/config/RBY1_A_v1_0.ros2_control.xacro (robot description, xacro)
@@ -1,5 +1,5 @@
 <?xml version="1.0"?>
 <robot xmlns:xacro="http://www.ros.org/wiki/xacro">
-    <xacro:macro name="RBY1_A_v1_0_ros2_control" params="name initial_positions_file use_fake_hardware:=true robot_ip:=127.0.0.1:50051 model:=a">
+    <xacro:macro name="RBY1_A_v1_0_ros2_control" params="name initial_positions_file use_fake_hardware:=true robot_ip:=127.0.0.1:50051 model:=a driver_namespace:=rby1">
         <xacro:property name="initial_positions" value="${xacro.load_yaml(initial_positions_file)['initial_positions']}"/>
 	      <xacro:arg name="robot_ip" default="127.0.0.1:50051" />
@@ -14,4 +14,5 @@
                     <param name="robot_ip">${robot_ip}</param>
                     <param name="model">${model}</param>
+                    <param name="driver_namespace">${driver_namespace}</param>
                 </xacro:unless>
             </hardware>

File: rby1_moveit/rby1_moveit_a_1_0/config/RBY1_A_v1_0.urdf.xacro (robot description, xacro)
@@ -7,4 +7,5 @@
     <xacro:arg name="model_name" default="rby1a" />
     <xacro:arg name="model_version" default="1_0" />
+    <xacro:arg name="driver_namespace" default="rby1" />
     <!-- Import RBY1_A_v1_0 urdf file -->
     <xacro:include filename="$(find rby1_description)/urdf/rby1a/model_v1_0.urdf" />
@@ -17,4 +18,5 @@
         robot_ip="$(arg robot_ip)"
         model="$(arg model)"
+        driver_namespace="$(arg driver_namespace)"
     />
 </robot>

File: rby1_moveit/rby1_moveit_a_1_1/config/RBY1_A_v1_1.ros2_control.xacro (robot description, xacro)
@@ -1,5 +1,5 @@
 <?xml version="1.0"?>
 <robot xmlns:xacro="http://www.ros.org/wiki/xacro">
-    <xacro:macro name="RBY1_A_v1_1_ros2_control" params="name initial_positions_file use_fake_hardware:=true robot_ip:=127.0.0.1:50051 model:=a">
+    <xacro:macro name="RBY1_A_v1_1_ros2_control" params="name initial_positions_file use_fake_hardware:=true robot_ip:=127.0.0.1:50051 model:=a driver_namespace:=rby1">
         <xacro:property name="initial_positions" value="${xacro.load_yaml(initial_positions_file)['initial_positions']}"/>
 	      <xacro:arg name="robot_ip" default="127.0.0.1:50051" />
@@ -14,4 +14,5 @@
                     <param name="robot_ip">${robot_ip}</param>
                     <param name="model">${model}</param>
+                    <param name="driver_namespace">${driver_namespace}</param>
                 </xacro:unless>
             </hardware>

File: rby1_moveit/rby1_moveit_a_1_1/config/RBY1_A_v1_1.urdf.xacro (robot description, xacro)
@@ -7,4 +7,5 @@
     <xacro:arg name="model_name" default="rby1a" />
     <xacro:arg name="model_version" default="1_1" />
+    <xacro:arg name="driver_namespace" default="rby1" />
     <!-- Import RBY1_A_v1_1 urdf file -->
     <xacro:include filename="$(find rby1_description)/urdf/rby1a/model_v1_1.urdf" />
@@ -17,4 +18,5 @@
         robot_ip="$(arg robot_ip)"
         model="$(arg model)"
+        driver_namespace="$(arg driver_namespace)"
     />
 </robot>

File: rby1_moveit/rby1_moveit_a_1_2/config/RBY1_A_v1_2.ros2_control.xacro (robot description, xacro)
@@ -1,5 +1,5 @@
 <?xml version="1.0"?>
 <robot xmlns:xacro="http://www.ros.org/wiki/xacro">
-    <xacro:macro name="RBY1_A_v1_2_ros2_control" params="name initial_positions_file use_fake_hardware:=true robot_ip:=127.0.0.1:50051 model:=a">
+    <xacro:macro name="RBY1_A_v1_2_ros2_control" params="name initial_positions_file use_fake_hardware:=true robot_ip:=127.0.0.1:50051 model:=a driver_namespace:=rby1">
         <xacro:property name="initial_positions" value="${xacro.load_yaml(initial_positions_file)['initial_positions']}"/>
 	      <xacro:arg name="robot_ip" default="127.0.0.1:50051" />
@@ -14,4 +14,5 @@
                     <param name="robot_ip">${robot_ip}</param>
                     <param name="model">${model}</param>
+                    <param name="driver_namespace">${driver_namespace}</param>
                 </xacro:unless>
             </hardware>

File: rby1_moveit/rby1_moveit_a_1_2/config/RBY1_A_v1_2.urdf.xacro (robot description, xacro)
@@ -7,4 +7,5 @@
     <xacro:arg name="model_name" default="rby1a" />
     <xacro:arg name="model_version" default="1_2" />
+    <xacro:arg name="driver_namespace" default="rby1" />
     <!-- Import RBY1_A_v1_2 urdf file -->
     <xacro:include filename="$(find rby1_description)/urdf/rby1a/model_v1_2.urdf" />
@@ -17,4 +18,5 @@
         robot_ip="$(arg robot_ip)"
         model="$(arg model)"
+        driver_namespace="$(arg driver_namespace)"
     />
 </robot>

File: rby1_moveit/rby1_moveit_m_1_0/config/RBY1_M_v1_0.ros2_control.xacro (robot description, xacro)
@@ -1,5 +1,5 @@
 <?xml version="1.0"?>
 <robot xmlns:xacro="http://www.ros.org/wiki/xacro">
-    <xacro:macro name="RBY1_M_v1_0_ros2_control" params="name initial_positions_file use_fake_hardware:=true robot_ip:=127.0.0.1:50051 model:=m">
+    <xacro:macro name="RBY1_M_v1_0_ros2_control" params="name initial_positions_file use_fake_hardware:=true robot_ip:=127.0.0.1:50051 model:=m driver_namespace:=rby1">
         <xacro:property name="initial_positions" value="${xacro.load_yaml(initial_positions_file)['initial_positions']}"/>
 	      <xacro:arg name="robot_ip" default="127.0.0.1:50051" />
@@ -14,4 +14,5 @@
                     <param name="robot_ip">${robot_ip}</param>
                     <param name="model">${model}</param>
+                    <param name="driver_namespace">${driver_namespace}</param>
                 </xacro:unless>
             </hardware>

File: rby1_moveit/rby1_moveit_m_1_0/config/RBY1_M_v1_0.urdf.xacro (robot description, xacro)
@@ -7,4 +7,5 @@
     <xacro:arg name="model_name" default="rby1m" />
     <xacro:arg name="model_version" default="1_0" />
+    <xacro:arg name="driver_namespace" default="rby1" />
     <!-- Import RBY1_M_v1_0 urdf file -->
     <xacro:include filename="$(find rby1_description)/urdf/rby1m/model_v1_0.urdf" />
@@ -17,4 +18,5 @@
         robot_ip="$(arg robot_ip)"
         model="$(arg model)"
+        driver_namespace="$(arg driver_namespace)"
     />
 </robot>

File: rby1_moveit/rby1_moveit_m_1_1/config/RBY1_M_v1_1.ros2_control.xacro (robot description, xacro)
@@ -1,5 +1,5 @@
 <?xml version="1.0"?>
 <robot xmlns:xacro="http://www.ros.org/wiki/xacro">
-    <xacro:macro name="RBY1_M_v1_1_ros2_control" params="name initial_positions_file use_fake_hardware:=true robot_ip:=127.0.0.1:50051 model:=m">
+    <xacro:macro name="RBY1_M_v1_1_ros2_control" params="name initial_positions_file use_fake_hardware:=true robot_ip:=127.0.0.1:50051 model:=m driver_namespace:=rby1">
         <xacro:property name="initial_positions" value="${xacro.load_yaml(initial_positions_file)['initial_positions']}"/>
 	      <xacro:arg name="robot_ip" default="127.0.0.1:50051" />
@@ -14,4 +14,5 @@
                     <param name="robot_ip">${robot_ip}</param>
                     <param name="model">${model}</param>
+                    <param name="driver_namespace">${driver_namespace}</param>
                 </xacro:unless>
             </hardware>

File: rby1_moveit/rby1_moveit_m_1_1/config/RBY1_M_v1_1.urdf.xacro (robot description, xacro)
@@ -7,4 +7,5 @@
     <xacro:arg name="model_name" default="rby1m" />
     <xacro:arg name="model_version" default="1_1" />
+    <xacro:arg name="driver_namespace" default="rby1" />
     <!-- Import RBY1_M_v1_1 urdf file -->
     <xacro:include filename="$(find rby1_description)/urdf/rby1m/model_v1_1.urdf" />
@@ -17,4 +18,5 @@
         robot_ip="$(arg robot_ip)"
         model="$(arg model)"
+        driver_namespace="$(arg driver_namespace)"
     />
 </robot>

File: rby1_moveit/rby1_moveit_m_1_2/config/RBY1_M_v1_2.ros2_control.xacro (robot description, xacro)
@@ -1,5 +1,5 @@
 <?xml version="1.0"?>
 <robot xmlns:xacro="http://www.ros.org/wiki/xacro">
-    <xacro:macro name="RBY1_M_v1_2_ros2_control" params="name initial_positions_file use_fake_hardware:=true robot_ip:=127.0.0.1:50051 model:=m">
+    <xacro:macro name="RBY1_M_v1_2_ros2_control" params="name initial_positions_file use_fake_hardware:=true robot_ip:=127.0.0.1:50051 model:=m driver_namespace:=rby1">
         <xacro:property name="initial_positions" value="${xacro.load_yaml(initial_positions_file)['initial_positions']}"/>
 	      <xacro:arg name="robot_ip" default="127.0.0.1:50051" />
@@ -14,4 +14,5 @@
                     <param name="robot_ip">${robot_ip}</param>
                     <param name="model">${model}</param>
+                    <param name="driver_namespace">${driver_namespace}</param>
                 </xacro:unless>
             </hardware>

File: rby1_moveit/rby1_moveit_m_1_2/config/RBY1_M_v1_2.urdf.xacro (robot description, xacro)
@@ -7,4 +7,5 @@
     <xacro:arg name="model_name" default="rby1m" />
     <xacro:arg name="model_version" default="1_2" />
+    <xacro:arg name="driver_namespace" default="rby1" />
     <!-- Import RBY1_M_v1_2 urdf file -->
     <xacro:include filename="$(find rby1_description)/urdf/rby1m/model_v1_2.urdf" />
@@ -17,4 +18,5 @@
         robot_ip="$(arg robot_ip)"
         model="$(arg model)"
+        driver_namespace="$(arg driver_namespace)"
     />
 </robot>

File: rby1_moveit/rby1_moveit_m_1_3/config/RBY1_M_v1_3.ros2_control.xacro (robot description, xacro)
@@ -1,5 +1,5 @@
 <?xml version="1.0"?>
 <robot xmlns:xacro="http://www.ros.org/wiki/xacro">
-    <xacro:macro name="RBY1_M_v1_3_ros2_control" params="name initial_positions_file use_fake_hardware:=true robot_ip:=127.0.0.1:50051 model:=m">
+    <xacro:macro name="RBY1_M_v1_3_ros2_control" params="name initial_positions_file use_fake_hardware:=true robot_ip:=127.0.0.1:50051 model:=m driver_namespace:=rby1">
         <xacro:property name="initial_positions" value="${xacro.load_yaml(initial_positions_file)['initial_positions']}"/>
 	      <xacro:arg name="robot_ip" default="127.0.0.1:50051" />
@@ -14,4 +14,5 @@
                     <param name="robot_ip">${robot_ip}</param>
                     <param name="model">${model}</param>
+                    <param name="driver_namespace">${driver_namespace}</param>
                 </xacro:unless>
             </hardware>

File: rby1_moveit/rby1_moveit_m_1_3/config/RBY1_M_v1_3.urdf.xacro (robot description, xacro)
@@ -7,4 +7,5 @@
     <xacro:arg name="model_name" default="rby1m" />
     <xacro:arg name="model_version" default="1_3" />
+    <xacro:arg name="driver_namespace" default="rby1" />
     <!-- Import RBY1_M_v1_3 urdf file -->
     <xacro:include filename="$(find rby1_description)/urdf/rby1m/model_v1_3.urdf" />
@@ -17,4 +18,5 @@
         robot_ip="$(arg robot_ip)"
         model="$(arg model)"
+        driver_namespace="$(arg driver_namespace)"
     />
 </robot>
