Commit message: update urdf

File: rby1_description/urdf/rby1a/model_v1_2.urdf (robot description, URDF)
Before this commit: robot RBY1_A_v1_2, 34 links, 33 joints
Joints:
- joint gripper_finger_r2_joint: mimic (none) -> joint=gripper_finger_r1_joint multiplier=1.0 offset=0.0

File: rby1_description/urdf/rby1m/model_v1_2.urdf (robot description, URDF)
Before this commit: robot RBY1_M_v1_2, 36 links, 35 joints
Joints:
- joint gripper_finger_r2_joint: mimic (none) -> joint=gripper_finger_r1_joint multiplier=1.0 offset=0.0
