Commit message: feat(description): command interfaces and gpios for all RB-Y1 modes
Joints export position (and stiffness/damping_ratio/torque_limit), wheels velocity;
gpio blocks declare gravity compensation, SE2 velocity, Cartesian, Cartesian impedance,
impedance and optimal control targets and a status block. Adds the gripper
ros2_control block and backend/rate/gripper xacro arguments.

Co-Authored-By: Claude Opus 5.5 <noreply@anthropic.com>

File: rby1_description/urdf/rby1a.urdf.xacro (robot description, xacro)
@@ -3,20 +3,38 @@
   <!--
     Top-level wrapper for the RBY1-A platform.
-    Supported versions: 1.0, 1.1, 1.2 (default).
-    Vendored from rby1-sdk/models/rby1a/urdf/model_v<version>.urdf.
+    Supported versions: 1.0, 1.1, 1.2 (default). Vendored from rby1-sdk/models/rby1a/urdf/model_v<version>.urdf.
   -->
   <xacro:arg name="version" default="1.2"/>
-  <xacro:arg name="robot_ip" default="127.0.0.1:50051"/>
+  <xacro:arg name="robot_ip" default="192.168.30.1:50051"/>
   <xacro:arg name="use_mock_hardware" default="false"/>
-  <xacro:arg name="auto_reconnect" default="true"/>
-  <xacro:arg name="read_timeout_sec" default="0.5"/>
-  <xacro:arg name="connect_timeout_sec" default="3.0"/>
+  <!-- sdk: real robot or rby1 simulator core; fake: in-memory robot for tests -->
+  <xacro:arg name="backend" default="sdk"/>
+  <xacro:arg name="auto_enable" default="false"/>
+  <xacro:arg name="command_rate" default="100"/>
+  <xacro:arg name="state_rate" default="200"/>
+  <xacro:arg name="impedance" default="true"/>
+  <xacro:arg name="task_space" default="true"/>
+  <xacro:arg name="gripper" default="false"/>
+  <xacro:arg name="gripper_backend" default="rb_dynamixel"/>
+  <xacro:arg name="gripper_device" default="/dev/rby1_gripper"/>
   <xacro:include filename="$(find rby1_description)/urdf/rby1a/v$(arg version)/model.xacro"/>
   <xacro:include filename="$(find rby1_description)/urdf/rby1.ros2_control.xacro"/>
+  <xacro:include filename="$(find rby1_description)/urdf/rby1_gripper.ros2_control.xacro"/>
   <xacro:rby1a_ros2_control
     robot_ip="$(arg robot_ip)"
     use_mock_hardware="$(arg use_mock_hardware)"
-    auto_reconnect="$(arg auto_reconnect)"
-    read_timeout_sec="$(arg read_timeout_sec)"
-    connect_timeout_sec="$(arg connect_timeout_sec)"/>
+    backend="$(arg backend)"
+    auto_enable="$(arg auto_enable)"
+    command_rate="$(arg command_rate)"
+    state_rate="$(arg state_rate)"
+    impedance="$(arg impedance)"
+    task_space="$(arg task_space)"/>
+  <xacro:if value="$(arg gripper)">
+    <xacro:rby1_gripper_ros2_control
+      robot_ip="$(arg robot_ip)"
+      model="a"
+      use_mock_hardware="$(arg use_mock_hardware)"
+      backend="$(arg gripper_backend)"
+      device="$(arg gripper_device)"/>
+  </xacro:if>
 </robot>

File: rby1_description/urdf/rby1m.urdf.xacro (robot description, xacro)
@@ -3,20 +3,38 @@
   <!--
     Top-level wrapper for the RBY1-M platform.
-    Supported versions: 1.0, 1.1, 1.2 (default), 1.3 (WY/WP/WR wrist).
-    Vendored from rby1-sdk/models/rby1m/urdf/model_v<version>.urdf.
+    Supported versions: 1.0, 1.1, 1.2 (default), 1.3 (WY/WP/WR wrist). Vendored from rby1-sdk/models/rby1m/urdf/model_v<version>.urdf.
   -->
   <xacro:arg name="version" default="1.2"/>
-  <xacro:arg name="robot_ip" default="127.0.0.1:50051"/>
+  <xacro:arg name="robot_ip" default="192.168.30.1:50051"/>
   <xacro:arg name="use_mock_hardware" default="false"/>
-  <xacro:arg name="auto_reconnect" default="true"/>
-  <xacro:arg name="read_timeout_sec" default="0.5"/>
-  <xacro:arg name="connect_timeout_sec" default="3.0"/>
+  <!-- sdk: real robot or rby1 simulator core; fake: in-memory robot for tests -->
+  <xacro:arg name="backend" default="sdk"/>
+  <xacro:arg name="auto_enable" default="false"/>
+  <xacro:arg name="command_rate" default="100"/>
+  <xacro:arg name="state_rate" default="200"/>
+  <xacro:arg name="impedance" default="true"/>
+  <xacro:arg name="task_space" default="true"/>
+  <xacro:arg name="gripper" default="false"/>
+  <xacro:arg name="gripper_backend" default="rb_dynamixel"/>
+  <xacro:arg name="gripper_device" default="/dev/rby1_gripper"/>
   <xacro:include filename="$(find rby1_description)/urdf/rby1m/v$(arg version)/model.xacro"/>
   <xacro:include filename="$(find rby1_description)/urdf/rby1.ros2_control.xacro"/>
+  <xacro:include filename="$(find rby1_description)/urdf/rby1_gripper.ros2_control.xacro"/>
   <xacro:rby1m_ros2_control
     robot_ip="$(arg robot_ip)"
     use_mock_hardware="$(arg use_mock_hardware)"
-    auto_reconnect="$(arg auto_reconnect)"
-    read_timeout_sec="$(arg read_timeout_sec)"
-    connect_timeout_sec="$(arg connect_timeout_sec)"/>
+    backend="$(arg backend)"
+    auto_enable="$(arg auto_enable)"
+    command_rate="$(arg command_rate)"
+    state_rate="$(arg state_rate)"
+    impedance="$(arg impedance)"
+    task_space="$(arg task_space)"/>
+  <xacro:if value="$(arg gripper)">
+    <xacro:rby1_gripper_ros2_control
+      robot_ip="$(arg robot_ip)"
+      model="m"
+      use_mock_hardware="$(arg use_mock_hardware)"
+      backend="$(arg gripper_backend)"
+      device="$(arg gripper_device)"/>
+  </xacro:if>
 </robot>

File: rby1_description/urdf/rby1ub.urdf.xacro (robot description, xacro)
@@ -5,16 +5,35 @@
     Single variant; vendored from rby1-sdk/models/rby1ub/urdf/model.urdf.
   -->
-  <xacro:arg name="robot_ip" default="127.0.0.1:50051"/>
-  <xacro:arg name="use_mock_hardware" default="true"/>
-  <xacro:arg name="auto_reconnect" default="true"/>
-  <xacro:arg name="read_timeout_sec" default="0.5"/>
-  <xacro:arg name="connect_timeout_sec" default="3.0"/>
+  <xacro:arg name="robot_ip" default="192.168.30.1:50051"/>
+  <xacro:arg name="use_mock_hardware" default="false"/>
+  <!-- sdk: real robot or rby1 simulator core; fake: in-memory robot for tests -->
+  <xacro:arg name="backend" default="sdk"/>
+  <xacro:arg name="auto_enable" default="false"/>
+  <xacro:arg name="command_rate" default="100"/>
+  <xacro:arg name="state_rate" default="200"/>
+  <xacro:arg name="impedance" default="true"/>
+  <xacro:arg name="task_space" default="true"/>
+  <xacro:arg name="gripper" default="false"/>
+  <xacro:arg name="gripper_backend" default="rb_dynamixel"/>
+  <xacro:arg name="gripper_device" default="/dev/rby1_gripper"/>
   <xacro:include filename="$(find rby1_description)/urdf/rby1ub/model.xacro"/>
   <xacro:include filename="$(find rby1_description)/urdf/rby1.ros2_control.xacro"/>
+  <xacro:include filename="$(find rby1_description)/urdf/rby1_gripper.ros2_control.xacro"/>
   <xacro:rby1ub_ros2_control
     robot_ip="$(arg robot_ip)"
     use_mock_hardware="$(arg use_mock_hardware)"
-    auto_reconnect="$(arg auto_reconnect)"
-    read_timeout_sec="$(arg read_timeout_sec)"
-    connect_timeout_sec="$(arg connect_timeout_sec)"/>
+    backend="$(arg backend)"
+    auto_enable="$(arg auto_enable)"
+    command_rate="$(arg command_rate)"
+    state_rate="$(arg state_rate)"
+    impedance="$(arg impedance)"
+    task_space="$(arg task_space)"/>
+  <xacro:if value="$(arg gripper)">
+    <xacro:rby1_gripper_ros2_control
+      robot_ip="$(arg robot_ip)"
+      model="ub"
+      use_mock_hardware="$(arg use_mock_hardware)"
+      backend="$(arg gripper_backend)"
+      device="$(arg gripper_device)"/>
+  </xacro:if>
 </robot>

Commit message: feat: SDK real-time control as the exclusive realtime mode
When a controller claims position, effort and feedback_gain of every torso and arm
joint (xacro realtime:=true, body_realtime_controller), the hardware closes the command
stream and runs Robot::Control on a backend thread. The 2 ms loop applies the robot's
fault rules (0.004 rad per tick, 0.15 rad tracking limit, gain 0-10, feedforward within
the URDF effort, wheels at rest, finish on stale state); on deactivation it finishes and
the stream resumes with a hold. Tested against the fake backend.

Co-Authored-By: Claude Opus 5.5 <noreply@anthropic.com>

File: rby1_description/urdf/rby1.ros2_control.xacro (robot description, xacro)
@@ -15,5 +15,5 @@
 <robot xmlns:xacro="http://www.ros.org/wiki/xacro">
   <!-- ===== joints ===================================================================== -->
-  <xacro:macro name="rby1_joint" params="name position:=true impedance:=false velocity:=false">
+  <xacro:macro name="rby1_joint" params="name position:=true impedance:=false velocity:=false realtime:=false">
     <joint name="${name}">
       <xacro:if value="${position}">
@@ -27,4 +27,8 @@
       <xacro:if value="${velocity}">
         <command_interface name="velocity"/>
+      </xacro:if>
+      <xacro:if value="${realtime}">
+        <command_interface name="effort"/>
+        <command_interface name="feedback_gain"/>
       </xacro:if>
       <state_interface name="position">
@@ -35,8 +39,10 @@
     </joint>
   </xacro:macro>
-  <xacro:macro name="rby1_joint_list" params="names position impedance velocity">
+  <xacro:macro name="rby1_joint_list" params="names position impedance velocity realtime:=false">
     <xacro:if value="${len(names) > 0}">
-      <xacro:rby1_joint name="${names[0]}" position="${position}" impedance="${impedance}" velocity="${velocity}"/>
-      <xacro:rby1_joint_list names="${names[1:]}" position="${position}" impedance="${impedance}" velocity="${velocity}"/>
+      <xacro:rby1_joint name="${names[0]}" position="${position}" impedance="${impedance}" velocity="${velocity}"
+        realtime="${realtime}"/>
+      <xacro:rby1_joint_list names="${names[1:]}" position="${position}" impedance="${impedance}" velocity="${velocity}"
+        realtime="${realtime}"/>
     </xacro:if>
   </xacro:macro>
@@ -190,8 +196,9 @@
       mobility:  export wheel velocity and base_se2
       task_space: export Cartesian, Cartesian impedance, impedance and optimal control gpios
+      realtime:  export effort and feedback_gain on torso, arm and head joints (SDK real-time control)
   -->
   <xacro:macro name="rby1_ros2_control"
     params="model torso_joints wheel_joints torso_link robot_ip use_mock_hardware backend:=sdk auto_enable:=false
-            command_rate:=100 state_rate:=200 impedance:=true task_space:=true name:=RBY1System">
+            command_rate:=100 state_rate:=200 impedance:=true task_space:=true realtime:=false name:=RBY1System">
     <xacro:property name="arm_r" value="${['right_arm_0', 'right_arm_1', 'right_arm_2', 'right_arm_3', 'right_arm_4', 'right_arm_5', 'right_arm_6']}"/>
     <xacro:property name="arm_l" value="${['left_arm_0', 'left_arm_1', 'left_arm_2', 'left_arm_3', 'left_arm_4', 'left_arm_5', 'left_arm_6']}"/>
@@ -199,8 +206,12 @@
       <xacro:rby1_hardware model="${model}" robot_ip="${robot_ip}" use_mock_hardware="${use_mock_hardware}"
         backend="${backend}" auto_enable="${auto_enable}" command_rate="${command_rate}" state_rate="${state_rate}"/>
-      <xacro:rby1_joint_list names="${torso_joints}" position="true" impedance="${impedance}" velocity="false"/>
-      <xacro:rby1_joint_list names="${arm_r}" position="true" impedance="${impedance}" velocity="false"/>
-      <xacro:rby1_joint_list names="${arm_l}" position="true" impedance="${impedance}" velocity="false"/>
-      <xacro:rby1_joint_list names="${['head_0', 'head_1']}" position="true" impedance="false" velocity="false"/>
+      <xacro:rby1_joint_list names="${torso_joints}" position="true" impedance="${impedance}" velocity="false"
+        realtime="${realtime}"/>
+      <xacro:rby1_joint_list names="${arm_r}" position="true" impedance="${impedance}" velocity="false"
+        realtime="${realtime}"/>
+      <xacro:rby1_joint_list names="${arm_l}" position="true" impedance="${impedance}" velocity="false"
+        realtime="${realtime}"/>
+      <xacro:rby1_joint_list names="${['head_0', 'head_1']}" position="true" impedance="false" velocity="false"
+        realtime="${realtime}"/>
       <xacro:rby1_joint_list names="${wheel_joints}" position="false" impedance="false" velocity="true"/>
       <xacro:rby1_gravity_compensation_gpio component="torso"/>
@@ -282,6 +293,6 @@
   <!-- Model wrappers (kept for compatibility with the earlier read-only description). -->
   <xacro:macro name="rby1a_ros2_control" params="robot_ip use_mock_hardware backend:=sdk auto_enable:=false
-      command_rate:=100 state_rate:=200 impedance:=true task_space:=true">
-    <xacro:rby1_ros2_control model="a" robot_ip="${robot_ip}" use_mock_hardware="${use_mock_hardware}"
+      command_rate:=100 state_rate:=200 impedance:=true task_space:=true realtime:=false">
+    <xacro:rby1_ros2_control model="a" realtime="${realtime}" robot_ip="${robot_ip}" use_mock_hardware="${use_mock_hardware}"
       backend="${backend}" auto_enable="${auto_enable}" command_rate="${command_rate}" state_rate="${state_rate}"
       impedance="${impedance}" task_space="${task_space}" torso_link="link_torso_5"
@@ -289,6 +300,6 @@
   </xacro:macro>
   <xacro:macro name="rby1m_ros2_control" params="robot_ip use_mock_hardware backend:=sdk auto_enable:=false
-      command_rate:=100 state_rate:=200 impedance:=true task_space:=true">
-    <xacro:rby1_ros2_control model="m" robot_ip="${robot_ip}" use_mock_hardware="${use_mock_hardware}"
+      command_rate:=100 state_rate:=200 impedance:=true task_space:=true realtime:=false">
+    <xacro:rby1_ros2_control model="m" realtime="${realtime}" robot_ip="${robot_ip}" use_mock_hardware="${use_mock_hardware}"
       backend="${backend}" auto_enable="${auto_enable}" command_rate="${command_rate}" state_rate="${state_rate}"
       impedance="${impedance}" task_space="${task_space}" torso_link="link_torso_5"
@@ -297,6 +308,6 @@
   </xacro:macro>
   <xacro:macro name="rby1ub_ros2_control" params="robot_ip use_mock_hardware backend:=sdk auto_enable:=false
-      command_rate:=100 state_rate:=200 impedance:=true task_space:=true">
-    <xacro:rby1_ros2_control model="ub" robot_ip="${robot_ip}" use_mock_hardware="${use_mock_hardware}"
+      command_rate:=100 state_rate:=200 impedance:=true task_space:=true realtime:=false">
+    <xacro:rby1_ros2_control model="ub" realtime="${realtime}" robot_ip="${robot_ip}" use_mock_hardware="${use_mock_hardware}"
       backend="${backend}" auto_enable="${auto_enable}" command_rate="${command_rate}" state_rate="${state_rate}"
       impedance="${impedance}" task_space="${task_space}" torso_link="link_torso_5"

File: rby1_description/urdf/rby1a.urdf.xacro (robot description, xacro)
@@ -15,4 +15,6 @@
   <xacro:arg name="impedance" default="true"/>
   <xacro:arg name="task_space" default="true"/>
+  <!-- SDK real-time control (UDP, 2 ms): exports effort and feedback_gain command interfaces -->
+  <xacro:arg name="realtime" default="false"/>
   <xacro:arg name="gripper" default="false"/>
   <xacro:arg name="gripper_backend" default="rb_dynamixel"/>
@@ -29,5 +31,6 @@
     state_rate="$(arg state_rate)"
     impedance="$(arg impedance)"
-    task_space="$(arg task_space)"/>
+    task_space="$(arg task_space)"
+    realtime="$(arg realtime)"/>
   <xacro:if value="$(arg gripper)">
     <xacro:rby1_gripper_ros2_control

File: rby1_description/urdf/rby1m.urdf.xacro (robot description, xacro)
@@ -15,4 +15,6 @@
   <xacro:arg name="impedance" default="true"/>
   <xacro:arg name="task_space" default="true"/>
+  <!-- SDK real-time control (UDP, 2 ms): exports effort and feedback_gain command interfaces -->
+  <xacro:arg name="realtime" default="false"/>
   <xacro:arg name="gripper" default="false"/>
   <xacro:arg name="gripper_backend" default="rb_dynamixel"/>
@@ -29,5 +31,6 @@
     state_rate="$(arg state_rate)"
     impedance="$(arg impedance)"
-    task_space="$(arg task_space)"/>
+    task_space="$(arg task_space)"
+    realtime="$(arg realtime)"/>
   <xacro:if value="$(arg gripper)">
     <xacro:rby1_gripper_ros2_control

File: rby1_description/urdf/rby1ub.urdf.xacro (robot description, xacro)
@@ -14,4 +14,6 @@
   <xacro:arg name="impedance" default="true"/>
   <xacro:arg name="task_space" default="true"/>
+  <!-- SDK real-time control (UDP, 2 ms): exports effort and feedback_gain command interfaces -->
+  <xacro:arg name="realtime" default="false"/>
   <xacro:arg name="gripper" default="false"/>
   <xacro:arg name="gripper_backend" default="rb_dynamixel"/>
@@ -28,5 +30,6 @@
     state_rate="$(arg state_rate)"
     impedance="$(arg impedance)"
-    task_space="$(arg task_space)"/>
+    task_space="$(arg task_space)"
+    realtime="$(arg realtime)"/>
   <xacro:if value="$(arg gripper)">
     <xacro:rby1_gripper_ros2_control

Commit message: fix(hardware_interface): reliable auto_enable and state timeout; simulator validation report
Found validating against the Isaac Sim core (rby1-sim-isaac 0.10.7, upstream sources):
- auto_enable sent servo-on before power had come up and powered up with the control
  manager enabled (which faults it). The driver now disables the control manager
  first and waits for power and servo to report on (enable_timeout, 10 s).
- The core pauses its state stream for ~0.1 s when a Cartesian impedance control
  starts; default state_timeout 0.1 -> 0.25 s, exposed as a xacro parameter.
- docs/VALIDATION.md: every controller in MuJoCo and Isaac Sim, Humble and Jazzy.
- tools/sim_validation: reset_sim.py enables only a powered robot; summarize.py.

Co-Authored-By: Claude Opus 5.5 <noreply@anthropic.com>

File: rby1_description/urdf/rby1.ros2_control.xacro (robot description, xacro)
@@ -167,5 +167,5 @@
   </xacro:macro>
   <!-- ===== hardware ==================================================================== -->
-  <xacro:macro name="rby1_hardware" params="model robot_ip use_mock_hardware backend auto_enable command_rate state_rate">
+  <xacro:macro name="rby1_hardware" params="model robot_ip use_mock_hardware backend auto_enable command_rate state_rate state_timeout:=0.25">
     <hardware>
       <xacro:if value="${use_mock_hardware}">
@@ -180,4 +180,7 @@
         <param name="command_rate">${command_rate}</param>
         <param name="state_rate">${state_rate}</param>
+        <!-- Stop when no robot state arrived for this long [s] (the simulator core pauses its state
+             stream for ~0.1 s when it starts a Cartesian impedance control). -->
+        <param name="state_timeout">${state_timeout}</param>
         <!-- Values validated on the real robot (100 Hz stream, rby1_lab deploy runtime). -->
         <param name="minimum_time">0.1</param>
